File: PCB/PCB V1/PCB V1.kicad_pcb (KiCad board)
At the start: 2 copper layers, 100 x 100 mm, 50 parts, among them J1 Screw_Terminal_01x03, J2 Screw_Terminal_01x03, J3 USB_B, J4 Conn_01x02_Pin, K1 Relay_SPDT, K2 Relay_SPDT, Q1 S8050, Q2 S8050, Q3 S8050, SW1 On/Off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

Commit message: .
Parts:
- removed AHT1: AHT10, Connector_Molex:Molex_KK-254_AE-6410-04A_1x04_P2.54mm_Vertical
- removed GND1, VCC1: Conn_01x01_Pin, Connector_PinHeader_2.54mm:PinHeader_1x01_P2.54mm_Vertical
- removed INA1: Sensor de Corriente, Connector_PinHeader_2.54mm:PinHeader_1x06_P2.54mm_Vertical
- added DISPLAY2: AHT10, Connector_Molex:Molex_KK-254_AE-6410-04A_1x04_P2.54mm_Vertical, F.Cu at (136.8, 88.7)
- added DISPLAY3: DISPLAY, Connector_Molex:Molex_KK-254_AE-6410-04A_1x04_P2.54mm_Vertical, F.Cu at (144.7, 88.7)
- D5, D7: footprint Connector_Molex:Molex_KK-254_AE-6410-02A_1x02_P2.54mm_Vertical -> LED_THT:LED_D5.0mm_Clear
- J4: footprint Connector_PinHeader_2.54mm:PinHeader_1x02_P2.54mm_Vertical -> Connector_Molex:Molex_KK-254_AE-6410-02A_1x02_P2.54mm_Vertical
- moved D6 180.5 mm to (81.9, 41.0)
- moved D8 179.9 mm to (81.9, 48.0)
- moved K2 179.7 mm to (76.2, 44.1), turned to -90 degrees
- moved J4 174.4 mm to (91.0, 94.5), turned to -90 degrees
- moved SW3 164.6 mm to (88.5, 73.0), turned to 180 degrees
- moved K1 163.6 mm to (76.2, 26.0), turned to -90 degrees
- moved D7 155.1 mm to (98.0, 65.5), turned to -90 degrees
- moved J1 154.6 mm to (54.0, 37.1), turned to 90 degrees
- moved R14 152.9 mm to (86.0, 81.0)
- moved J2 151.5 mm to (54.0, 55.1), turned to 90 degrees
- moved R13 146.1 mm to (79.0, 79.0), turned to -90 degrees
- moved D5 141.0 mm to (105.0, 65.5), turned to -90 degrees
- moved D3 137.5 mm to (127.5, 118.0)
- moved R9 137.5 mm to (88.0, 57.9), turned to -90 degrees
- moved Q2 133.1 mm to (100.5, 61.0)
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Connections:
- ESP-1 pad 10: BOTON-B -> unconnected-(ESP-1-IO32-Pad10)
- ESP-1 pad 11: unconnected-(ESP-1-IO35-Pad11) -> RELE-B
- ESP-1 pad 12: unconnected-(ESP-1-IO34-Pad12) -> RELE-A
- ESP-1 pad 13: unconnected-(ESP-1-IO39-Pad13) -> BOTON-B
- ESP-1 pad 16: unconnected-(ESP-1-IO23-Pad16) -> BOTON-A
- ESP-1 pad 19: LED-A2 -> unconnected-(ESP-1-IO3-Pad19)
- ESP-1 pad 21: RELE-A -> unconnected-(ESP-1-IO19-Pad21)
- ESP-1 pad 22: RELE-B -> unconnected-(ESP-1-IO18-Pad22)
- ESP-1 pad 24: PUERTA -> unconnected-(ESP-1-IO17-Pad24)
- ESP-1 pad 28: unconnected-(ESP-1-IO15-Pad28) -> LED-A2
- ESP-1 pad 8: unconnected-(ESP-1-IO25-Pad8) -> PUERTA
- ESP-1 pad 9: BOTON-A -> unconnected-(ESP-1-IO33-Pad9)
Routing:
- net +3.3V: track 50.5 -> 331.0 mm, vias 0 -> 2
- net GND: track 184.8 -> 444.8 mm, vias 0 -> 6
- net Net-(D6-A): track 0.00 -> 56.9 mm
- net Net-(D8-A): track 0.00 -> 40.3 mm
- net LED-A2: track 0.00 -> 39.0 mm
- net RELE-B: track 0.00 -> 36.8 mm
- net BOTON-A: track 0.00 -> 28.2 mm
- net BOTON-B: track 0.00 -> 27.2 mm
- net PUERTA: track 0.00 -> 25.7 mm
- net RELE-A: track 0.00 -> 25.7 mm
- net LED-B2: track 0.00 -> 24.8 mm
- net Net-(J2-Pin_2): track 0.00 -> 24.2 mm
- net Net-(J1-Pin_2): track 0.00 -> 24.2 mm
- net Net-(Q3-B): track 0.00 -> 22.8 mm
- net Net-(Q1-B): track 0.00 -> 17.3 mm
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Other:
- board text added: "${REFERENCE}"
- board text added: "EITAN CHERNIAK URIEL DIGESTANI AARON YABRA"

Commit message: Update PCB V1.kicad_pcb
Parts:
- moved Cooler1 65.4 mm to (54.0, 61.5), turned to -90 degrees
Connections:
- Cooler1 pad 1: +5V -> NO
- J2 pad 1: Net-(J2-Pin_1) -> NO
- J2 pad 2: Net-(J2-Pin_2) -> +5V
- K2 pad 11: Net-(J2-Pin_2) -> +5V
- K2 pad 12: Net-(J2-Pin_1) -> NO
Routing:
- net +5V: track 94.1 -> 146.9 mm, vias 0 -> 2
- net Net-(J2-Pin_2): track 24.2 -> 0.00 mm
- net NO: track 0.00 -> 16.8 mm
- net Net-(J2-Pin_1): track 10.4 -> 0.00 mm
- net GND: track 444.8 -> 452.3 mm

Commit message: .
Parts:
- added ?: , , F.Cu at (85.1, 114.5)
- added ?: , , F.Cu at (97.0, 27.0)
- added GND1: Conn_01x01_Pin, Connector_PinHeader_2.54mm:PinHeader_1x01_P2.54mm_Vertical, F.Cu at (65.5, 68.5)
- added VCC1: Conn_01x01_Pin, Connector_PinHeader_2.54mm:PinHeader_1x01_P2.54mm_Vertical, F.Cu at (74.0, 88.5)
- moved D8 3.50 mm to (85.4, 48.0)
Connections:
- J2 pad 2: +5V -> Net-(J2-Pin_2)
- K2 pad 11: +5V -> Net-(J2-Pin_2)
Routing:
- net +5V: track 146.9 -> 83.6 mm, vias 2 -> 0
- net Net-(J2-Pin_2): track 0.00 -> 24.2 mm
- net GND: track 452.3 -> 470.4 mm
- net +3.3V: track 331.0 -> 337.0 mm

Commit message: .
Parts:
- removed D10: 1N4007, Diode_THT:D_DO-41_SOD81_P10.16mm_Horizontal
- R11: value 1.01K -> 20K
Connections:
- DISPLAY1 pad 2: +3.3V -> +5V
- J2 pad 2: Net-(J2-Pin_2) -> +5V
- K2 pad 11: Net-(J2-Pin_2) -> +5V
Routing:
- net +5V: track 83.6 -> 107.8 mm
- net Net-(J2-Pin_2): track 24.2 -> 0.00 mm
- net +3.3V: track 337.0 -> 328.4 mm

Commit message: .
Parts:
- R11: value 20K -> 22K
Changed lines of the file:
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@@
 			)
 		)
-		(property "Value" "20K"
+		(property "Value" "22K"
 			(at 5.08 2.37 90)
 			(layer "F.Fab")

Commit message: .
Parts:
- removed ? (x2): , 
- added C4: 100uF, Capacitor_THT:CP_Radial_D10.0mm_P3.50mm, F.Cu at (99.2, 103.3)
- added C5: 10uF, Capacitor_THT:CP_Radial_D5.0mm_P2.50mm, F.Cu at (94.9, 118.2)
- added C6: 100uf, Capacitor_THT:C_Disc_D7.5mm_W4.4mm_P5.00mm, F.Cu at (113.0, 121.0)
- added Cooler2: Bateria, TerminalBlock:TerminalBlock_bornier-2_P5.08mm, F.Cu at (96.2, 94.5)
- added R17: 560, Resistor_THT:R_Axial_DIN0207_L6.3mm_D2.5mm_P10.16mm_Horizontal, F.Cu at (108.7, 110.4)
- added R18: 330, Resistor_THT:R_Axial_DIN0207_L6.3mm_D2.5mm_P10.16mm_Horizontal, F.Cu at (108.7, 114.0)
- added U2: LM317_TO-220, Package_TO_SOT_THT:TO-220F-3_Vertical, F.Cu at (105.8, 118.6)
- R1, R7: value R_US -> 100
- R10, R9: value R_US -> 10K
- R12: value R_LDR -> 10K
- R2, R4: value R_US -> 1.6
- SW1: footprint Button_Switch_THT:SW_Slide_SPDT_Straight_CK_OS102011MS2Q -> TerminalBlock:TerminalBlock_bornier-2_P5.08mm
- moved GND1 213.5 mm to (278.9, 74.1)
- moved VCC1 205.1 mm to (278.9, 78.7)
- moved K2 189.4 mm to (265.5, 47.8), turned to 0 degrees
- moved D6 189.1 mm to (235.8, 150.9)
- moved D8 184.7 mm to (235.8, 155.2)
- moved D7 179.5 mm to (277.5, 68.0), turned to 0 degrees
- moved R14 176.8 mm to (262.7, 76.0)
- moved K1 173.8 mm to (248.7, 47.8), turned to 0 degrees
- moved Q2 170.4 mm to (267.0, 96.8)
- moved J1 165.9 mm to (206.8, 101.6), turned to 0 degrees
- moved D5 165.0 mm to (270.0, 68.0), turned to 0 degrees
- moved J2 162.6 mm to (206.8, 110.6), turned to 0 degrees
- moved Q1 160.7 mm to (267.0, 91.0), turned to 0 degrees
- moved D3 144.1 mm to (262.7, 68.1)
- moved R7 142.4 mm to (234.4, 70.2), turned to 0 degrees
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Connections:
- Cooler1 pad 1: NO -> +5V
- D5 pad 2: RELE-B -> +3.3V
- D7 pad 2: RELE-A -> +3.3V
- D9 pad 1: Net-(D9-K) -> +5VANTESDELLAVE
- J2 pad 2: +5V -> Net-(J2-Pin_2)
- J3 pad 1: Net-(D9-A) -> +5VANTESDELLAVE
- K2 pad 11: +5V -> Net-(J2-Pin_2)
- R1 pad 2: GND -> Net-(D6-A)
- R7 pad 2: GND -> Net-(D8-A)
- SW1 pad 1: Net-(D9-K) -> +5VANTESDELLAVE
Routing:
- net +3.3V: track 328.4 -> 51.9 mm, vias 2 -> 0
- net GND: track 470.4 -> 262.1 mm, vias 6 -> 0
- net Net-(D6-A): track 56.9 -> 0.00 mm
- net +5V: track 107.8 -> 57.0 mm
- net Net-(D8-A): track 40.3 -> 0.00 mm
- net LED-A2: track 39.0 -> 0.00 mm
- net RELE-B: track 36.8 -> 3.17 mm
- net +12V: track 0.00 -> 32.9 mm
- net BOTON-A: track 28.2 -> 0.00 mm
- net +5VANTESDELLAVE: track 0.00 -> 27.8 mm
- net SDA: track 27.5 -> 0.00 mm
- net LED-B2: track 24.8 -> 0.00 mm
- net Net-(J1-Pin_2): track 24.2 -> 0.00 mm
- net SCL: track 23.0 -> 0.00 mm
- net BOTON-B: track 27.2 -> 7.83 mm
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Other:
- board text removed: "${REFERENCE}"
- board text removed: "EITAN CHERNIAK URIEL DIGESTANI AARON YABRA"

Commit message: .
Parts:
- removed GND1, VCC1: Conn_01x01_Pin, Connector_PinHeader_2.54mm:PinHeader_1x01_P2.54mm_Vertical
- added D10: 1N4007, Diode_THT:D_DO-41_SOD81_P10.16mm_Horizontal, F.Cu at (182.5, 115.4)
- C3, C6: moved to B.Cu
- moved D3 123.2 mm to (141.5, 46.0), turned to 180 degrees
- moved D1 120.5 mm to (130.0, 46.0), turned to 180 degrees
- moved DISPLAY3 115.0 mm to (165.1, 45.8), turned to 180 degrees
- moved R14 111.3 mm to (154.5, 102.0), turned to 90 degrees
- moved SW2 111.2 mm to (151.0, 46.0)
- moved DISPLAY2 104.8 mm to (165.1, 53.6), turned to 180 degrees
- moved R2 101.1 mm to (133.5, 56.0), turned to 90 degrees
- moved DISPLAY1 96.1 mm to (165.1, 61.5), turned to 180 degrees
- moved R4 88.9 mm to (145.5, 56.1), turned to 90 degrees
- moved J3 83.3 mm to (185.2, 129.4)
- moved R6 81.1 mm to (230.8, 65.7), turned to 0 degrees
- moved Cooler2 80.6 mm to (167.0, 133.0), turned to 0 degrees
- moved SW1 78.4 mm to (189.5, 116.0), turned to 90 degrees
- moved C6 76.5 mm to (189.5, 120.5), turned to -90 degrees
- moved ESP-1 76.2 mm to (196.9, 68.3), turned to -90 degrees
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Connections:
- ESP-1 pad 13: BOTON-B -> unconnected-(ESP-1-IO39-Pad13)
- ESP-1 pad 18: LED-A1 -> unconnected-(ESP-1-IO1-Pad18)
- ESP-1 pad 21: unconnected-(ESP-1-IO19-Pad21) -> BOTON-B
- ESP-1 pad 22: unconnected-(ESP-1-IO18-Pad22) -> PUERTA
- ESP-1 pad 23: BUZZER -> LED-A2
- ESP-1 pad 24: unconnected-(ESP-1-IO17-Pad24) -> LED-A1
- ESP-1 pad 27: LED-B1 -> unconnected-(ESP-1-IO2-Pad27)
- ESP-1 pad 28: LED-A2 -> LED-B1
- ESP-1 pad 7: unconnected-(ESP-1-IO26-Pad7) -> BUZZER
- ESP-1 pad 8: PUERTA -> unconnected-(ESP-1-IO25-Pad8)
- J3 pad 1: +5VANTESDELLAVE -> Net-(D10-A)
Routing:
- net +3.3V: track 51.9 -> 192.4 mm, vias 0 -> 2
- net +5V: track 57.0 -> 147.7 mm, vias 0 -> 2
- net GND: track 262.1 -> 340.0 mm
- net LED-A1: track 0.00 -> 73.6 mm
- net LED-A2: track 0.00 -> 61.3 mm
- net BUZZER: track 0.00 -> 59.4 mm
- net BOTON-A: track 0.00 -> 27.9 mm
- net SDA: track 0.00 -> 24.9 mm
- net SCL: track 0.00 -> 24.8 mm
- net LED-B2: track 0.00 -> 17.5 mm
- net BOTON-B: track 7.83 -> 22.9 mm
- net PUERTA: track 8.75 -> 23.8 mm
- net +5VANTESDELLAVE: track 27.8 -> 16.1 mm
- net +12V: track 32.9 -> 43.5 mm
- net Net-(D2-K): track 0.00 -> 9.72 mm
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