File: PCB/PCB V1/PCB V1.kicad_pcb (KiCad board)
At the start: 2 copper layers, 100 x 100 mm, 55 parts, among them J1 Screw_Terminal_01x03, J2 Screw_Terminal_01x03, J3 USB_B, J4 Conn_01x02_Pin, K1 Relay_SPDT, K2 Relay_SPDT, Q1 S8050, Q2 S8050, Q3 S8050, SW1 On/Off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

Commit message: .
Parts:
- U1, U2: footprint Package_TO_SOT_THT:TO-220F-3_Vertical -> Package_TO_SOT_THT:TO-92_Inline
- moved D7 15.3 mm to (139.7, 80.0)
- moved R10 11.2 mm to (160.0, 83.8), turned to 90 degrees
- moved D8 1.27 mm to (133.3, 86.4)
Connections:
- ESP-1 pad 11: unconnected-(ESP-1-IO35-Pad11) -> LDR
- ESP-1 pad 14: LDR -> unconnected-(ESP-1-IO36-Pad14)
Routing:
- net GND: track 444.2 -> 423.7 mm
- net +3.3V: track 457.7 -> 438.8 mm, vias 6 -> 4
- net Net-(D7-K): track 3.81 -> 18.1 mm
- net BOTON-A: track 27.9 -> 35.3 mm
- net LDR: track 19.1 -> 22.6 mm
- net +5V: track 214.9 -> 217.6 mm, vias 4 -> 2
- net +12V: track 43.5 -> 46.1 mm
- net Net-(D9-A): track 35.7 -> 35.1 mm

Commit message: .
Parts:
- C3, C6: moved to F.Cu
- moved BZ1 170.9 mm to (254.0, 33.0), turned to 0 degrees
- moved Q3 162.7 mm to (256.5, 42.2), turned to 0 degrees
- moved R11 161.6 mm to (258.2, 45.9), turned to 180 degrees
- moved C5 130.7 mm to (276.9, 88.9)
- moved J2 124.2 mm to (219.7, 111.7), turned to 180 degrees
- moved C4 112.9 mm to (275.6, 100.3), turned to 180 degrees
- moved Cooler2 107.2 mm to (271.8, 110.5)
- moved Cooler1 105.8 mm to (259.1, 20.3), turned to 180 degrees
- moved C3 102.9 mm to (228.6, 110.5), turned to 0 degrees
- moved R17 101.9 mm to (261.6, 93.0), turned to 0 degrees
- moved R18 101.9 mm to (261.6, 88.9), turned to 0 degrees
- moved R15 99.2 mm to (233.7, 97.8), turned to 90 degrees
- moved J1 98.7 mm to (197.6, 112.0), turned to 180 degrees
- moved U2 96.8 mm to (264.2, 97.8)
- moved R1 93.8 mm to (201.4, 73.9), turned to -90 degrees
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Connections:
- ESP-1 pad 12: RELE-A -> RELE-B
- ESP-1 pad 13: RELE-B -> RELE-A
- ESP-1 pad 21: BOTON-B -> BUZZER
- ESP-1 pad 22: PUERTA -> LED-B2
- ESP-1 pad 24: LED-A1 -> LED-B1
- ESP-1 pad 25: unconnected-(ESP-1-IO16-Pad25) -> LED-A1
- ESP-1 pad 26: LED-B2 -> PUERTA
- ESP-1 pad 28: LED-B1 -> unconnected-(ESP-1-IO15-Pad28)
- ESP-1 pad 7: BUZZER -> BOTON-B
Routing:
- net +3.3V: track 438.8 -> 239.1 mm, vias 4 -> 0
- net +5V: track 217.6 -> 95.0 mm, vias 2 -> 0
- net GND: track 423.7 -> 304.6 mm, vias 4 -> 0
- net BUZZER: track 59.4 -> 6.16 mm
- net LED-B1: track 7.84 -> 58.2 mm
- net RELE-B: track 21.5 -> 64.3 mm
- net LED-B2: track 17.5 -> 42.4 mm
- net +12V: track 46.1 -> 22.1 mm
- net BOTON-A: track 35.3 -> 14.0 mm
- net PUERTA: track 23.8 -> 3.81 mm
- net BOTON-B: track 22.9 -> 3.81 mm
- net LDR: track 22.6 -> 3.81 mm
- net Net-(D8-A): track 20.9 -> 37.9 mm
- net Net-(D6-A): track 19.5 -> 34.1 mm
- net LED-A2: track 61.3 -> 50.1 mm
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- removed copper zone on B.Cu, net GND
Other:
- board outline removed
- board text removed: "GRUPO ¿?"

Commit message: .
Parts:
- moved R12 17.1 mm to (188.0, 63.5)
- moved J4 10.2 mm to (188.0, 52.7)
- moved R13 10.2 mm to (198.1, 46.4)
- moved D1 5.08 mm to (214.6, 36.8)
- moved D2 5.08 mm to (221.0, 36.8)
- moved D3 5.08 mm to (227.3, 36.8)
- moved D4 5.08 mm to (233.7, 36.8)
- moved R2 5.08 mm to (214.6, 21.6)
- moved R3 5.08 mm to (221.0, 21.6)
- moved R4 5.08 mm to (227.3, 21.6)
- moved R5 5.08 mm to (233.7, 21.6)
- moved R14 4.45 mm to (188.0, 57.1), turned to -90 degrees
- moved BZ1 2.54 mm to (256.5, 33.0)
- moved Q3 2.54 mm to (259.0, 42.2)
- moved R11 2.54 mm to (260.7, 45.9)
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Connections:
- ESP-1 pad 10: unconnected-(ESP-1-IO32-Pad10) -> BOTON-A
- ESP-1 pad 16: BOTON-A -> unconnected-(ESP-1-IO23-Pad16)
- ESP-1 pad 26: PUERTA -> unconnected-(ESP-1-IO4-Pad26)
- ESP-1 pad 7: BOTON-B -> PUERTA
- ESP-1 pad 9: unconnected-(ESP-1-IO33-Pad9) -> BOTON-B
Routing:
- net GND: track 304.6 -> 496.3 mm, vias 0 -> 4
- net PUERTA: track 3.81 -> 117.6 mm
- net +3.3V: track 239.1 -> 334.1 mm, vias 0 -> 2
- net BOTON-B: track 3.81 -> 94.7 mm
- net LDR: track 3.81 -> 71.8 mm
- net +5V: track 95.0 -> 157.8 mm
- net BOTON-A: track 14.0 -> 71.5 mm
- net LED-B2: track 42.4 -> 36.2 mm
- net LED-A1: track 67.5 -> 61.5 mm
- net LED-A2: track 50.1 -> 44.7 mm
- net LED-B1: track 58.2 -> 53.3 mm
- net SDA: track 32.4 -> 31.4 mm
- net SCL: track 30.9 -> 29.8 mm
- net BUZZER: track 6.16 -> 5.10 mm
- added copper zone on B.Cu, net GND
Other:
- board outline added: 100 x 100 mm

Commit message: .
Parts:
- added GND1: Conn_01x01_Pin, Connector_PinHeader_2.54mm:PinHeader_1x01_P2.54mm_Vertical, F.Cu at (268.7, 39.5)
- added VCC1: Conn_01x01_Pin, Connector_PinHeader_2.54mm:PinHeader_1x01_P2.54mm_Vertical, F.Cu at (278.4, 38.3)
Connections:
- net NO renamed Net-(J2-Pin_1)
Routing:
- net GND: track 496.3 -> 526.7 mm, vias 4 -> 6
- net +5V: track 157.8 -> 163.4 mm
- net +3.3V: track 334.1 -> 335.6 mm
- net (no net): vias 0 -> 2
Other:
- board text added: "GRUPO8"
