File: PCB/PCB V1/PCB V1.kicad_pcb (KiCad board)
At the start: 2 copper layers, 100 x 100 mm, 56 parts, among them J1 Screw_Terminal_01x03, J2 Screw_Terminal_01x03, J3 USB_B, J4 Conn_01x02_Pin, K1 Relay_SPDT, K2 Relay_SPDT, Q1 S8050, Q2 S8050, Q3 S8050, SW1 On/Off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

Commit message: .
Changed lines of the file:
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@@
 		(tags "Resistor Axial_DIN0207 series Axial Horizontal pin pitch 10.16mm 0.25W = 1/4W length 6.3mm diameter 2.5mm")
 		(property "Reference" "R18"
-			(at 5.08 -2.37 0)
+			(at 11.888358 -0.050262 90)
 			(layer "F.SilkS")
 			(effects
@@
 		(tags "connector Molex KK-254 vertical")
 		(property "Reference" "DISPLAY3"
-			(at 3.81 -4.12 180)
+			(at -2.54 0.23 -90)
 			(layer "F.SilkS")
 			(effects
@@
 		(tags "to-92 sc-43 sc-43a sot54 PA33 transistor")
 		(property "Reference" "Q2"
-			(at 1.27 -3.56 0)
+			(at 5.08 0.06 90)
 			(layer "F.SilkS")
 			(effects
@@
 		(tags "Resistor Axial_DIN0207 series Axial Horizontal pin pitch 10.16mm 0.25W = 1/4W length 6.3mm diameter 2.5mm")
 		(property "Reference" "R12"
-			(at 5.08 -2.37 0)
+			(at 10.16 2.54 90)
 			(layer "F.SilkS")
 			(effects
@@
 		(tags "Through hole pin header THT 1x01 2.54mm single row")
 		(property "Reference" "GND1"
-			(at 0 -2.33 0)
+			(at 3.0988 -0.127 90)
 			(layer "F.SilkS")
 			(effects
@@
 		(tags "connector Molex KK-254 vertical")
 		(property "Reference" "D2"
-			(at 1.27 -4.12 0)
+			(at 1.27 5.08 90)
 			(layer "F.SilkS")
 			(effects
@@
 		(tags "Diode DO-41_SOD81 series Axial Horizontal pin pitch 10.16mm  length 5.2mm diameter 2.7mm")
 		(property "Reference" "D8"
-			(at 5.08 -2.47 0)
+			(at -2.54 0.06 90)
 			(layer "F.SilkS")
 			(effects
@@
 		(tags "terminal block bornier3")
 		(property "Reference" "J2"
-			(at 5.05 -4.65 180)
+			(at -3.81 -0.06 -90)
 			(layer "F.SilkS")
 			(effects
@@
 		(tags "to-92 sc-43 sc-43a sot54 PA33 transistor")
 		(property "Reference" "Q3"
-			(at 1.27 -3.56 0)
+			(at 5.160296 -0.330072 90)
 			(layer "F.SilkS")
 			(effects
@@
 		(tags "to-92 sc-43 sc-43a sot54 PA33 transistor")
 		(property "Reference" "U2"
-			(at 1.27 -3.56 0)
+			(at -2.54 0 90)
 			(layer "F.SilkS")
 			(effects
@@
 		(tags "Resistor Axial_DIN0207 series Axial Horizontal pin pitch 10.16mm 0.25W = 1/4W length 6.3mm diameter 2.5mm")
 		(property "Reference" "R16"
-			(at 5.08 -2.37 90)
+			(at 5.08 2.54 90)
 			(layer "F.SilkS")
 			(effects
@@
 		(tags "connector Molex KK-254 vertical")
 		(property "Reference" "DISPLAY2"
-			(at 3.81 -4.12 180)
+			(at -2.54 0 -90)
 			(layer "F.SilkS")
 			(effects
@@
 			)
 		)
-		(sheetname "Raíz")
-		(sheetfile "PCB V1.kicad_sch")
 		(attr through_hole)
 		(fp_line
@@
 			(layer "F.SilkS")
 		)
+		(fp_rect
+			(start 0 -0.18)
+			(end 28 51.02)
+			(stroke
+				(width 0.05)
+				(type default)
+			)
+			(fill none)
+			(layer "F.CrtYd")
+		)
 		(pad "1" thru_hole circle
 			(at 26.67 8.89 270)
@@
 		(tags "Diode DO-41_SOD81 series Axial Horizontal pin pitch 10.16mm  length 5.2mm diameter 2.7mm")
 		(property "Reference" "D9"
-			(at 5.08 -2.47 0)
+			(at 5.08 2.54 90)
 			(layer "F.SilkS")
 			(effects
@@
 		(tags "spdt relay")
 		(property "Reference" "K1"
-			(at 6 -4.2 0)
+			(at 15.81 8.105 90)
 			(layer "F.SilkS")
 			(effects
@@
 		(tags "LED diameter 5.0mm 2 pins")
 		(property "Reference" "D5"
-			(at 1.27 -3.96 180)
+			(at -3.11 0.285 -90)
 			(layer "F.SilkS")
 			(effects
@@
 		(tags "terminal block bornier2")
 		(property "Reference" "Cooler1"
-			(at 2.54 -5.08 180)
+			(at -3.81 -0.21 -90)
 			(layer "F.SilkS")
 			(effects
@@
 		(tags "connector Molex KK-254 vertical")
 		(property "Reference" "D3"
-			(at 1.27 -4.12 0)
+			(at 1.27 5.08 90)
 			(layer "F.SilkS")
 			(effects
@@
 		(tags "buzzer")
 		(property "Reference" "BZ1"
-			(at 3.8 -7.2 0)
+			(at 11.43 0 90)
 			(layer "F.SilkS")
 			(effects
@@
 		(tags "connector Molex KK-254 vertical")
 		(property "Reference" "DISPLAY1"
-			(at 3.81 -4.12 180)
+			(at 10.16 -0.23 -90)
 			(layer "F.SilkS")
 			(effects
@@
 		(tags "Resistor Axial_DIN0207 series Axial Horizontal pin pitch 10.16mm 0.25W = 1/4W length 6.3mm diameter 2.5mm")
 		(property "Reference" "R10"
-			(at 5.08 -2.37 0)
+			(at 12.887245 0.031169 90)
 			(layer "F.SilkS")
 			(effects
@@
 		(tags "connector Molex KK-254 vertical")
 		(property "Reference" "D4"
-			(at 1.27 -4.12 0)
+			(at 1.27 5.08 90)
 			(layer "F.SilkS")
 			(effects
@@
 		(tags "Through hole pin header THT 1x01 2.54mm single row")
 		(property "Reference" "VCC1"
-			(at 0 -2.33 0)
+			(at 2.2606 -0.2032 90)
 			(layer "F.SilkS")
 			(effects
@@
 		(tags "C Disc series Radial pin pitch 5.00mm  diameter 7.5mm width 4.4mm Capacitor")
 		(property "Reference" "C3"
-			(at 2.5 -3.45 0)
+			(at -2.58 0 90)
 			(layer "F.SilkS")
 			(effects
@@
 		(tags "terminal block bornier3")
 		(property "Reference" "J1"
-			(at 5.05 -4.65 180)
+			(at -4.38 0.285 -90)
 			(layer "F.SilkS")
 			(effects
@@
 		(tags "C Disc series Radial pin pitch 5.00mm  diameter 7.5mm width 4.4mm Capacitor")
 		(property "Reference" "C6"
-			(at 2.5 -3.45 0)
+			(at 7.62 0 90)
 			(layer "F.SilkS")
 			(effects
@@
 		(tags "spdt relay")
 		(property "Reference" "K2"
-			(at 6 -4.2 0)
+			(at 14.54 7.18 90)
 			(layer "F.SilkS")
 			(effects
@@
 		(tags "to-92 sc-43 sc-43a sot54 PA33 transistor")
 		(property "Reference" "Q1"
-			(at 1.27 -3.56 0)
+			(at 4.38 -0.285 90)
 			(layer "F.SilkS")
 			(effects
@@
 		(tags "Resistor Axial_DIN0207 series Axial Horizontal pin pitch 10.16mm 0.25W = 1/4W length 6.3mm diameter 2.5mm")
 		(property "Reference" "R15"
-			(at 5.08 -2.37 -90)
+			(at 6.35 2.54 -90)
 			(layer "F.SilkS")
 			(effects
@@
 		(tags "USB-B receptacle horizontal through-hole")
 		(property "Reference" "J3"
-			(at 6.76 -7.77 90)
+			(at -0.002785 -6.492326 90)
 			(layer "F.SilkS")
 			(effects
@@
 		(tags "connector Molex KK-254 vertical")
 		(property "Reference" "D1"
-			(at 1.27 -4.12 0)
+			(at 1.27 5.08 90)
 			(layer "F.SilkS")
 			(effects
@@
 		(tags "Diode DO-41_SOD81 series Axial Horizontal pin pitch 10.16mm  length 5.2mm diameter 2.7mm")
 		(property "Reference" "D6"
-			(at 5.08 -2.47 0)
+			(at -2.682371 -0.031879 90)
 			(layer "F.SilkS")
 			(effects
@@
 		(tags "LED diameter 5.0mm 2 pins")
 		(property "Reference" "D7"
-			(at 1.27 -3.96 180)
+			(at -2.54 -0.06 -90)
 			(layer "F.SilkS")
 			(effects
@@
 		(tags "Resistor Axial_DIN0207 series Axial Horizontal pin pitch 10.16mm 0.25W = 1/4W length 6.3mm diameter 2.5mm")
 		(property "Reference" "R11"
-			(at 5.08 -2.37 180)
+			(at -2.181788 0.179106 -90)
 			(layer "F.SilkS")
 			(effects
@@
 		(tags "terminal block bornier2")
 		(property "Reference" "SW1"
-			(at 2.54 -5.08 180)
+			(at 8.89 0 -90)
 			(layer "F.SilkS")
 			(effects
@@
 		(tags "Resistor Axial_DIN0207 series Axial Horizontal pin pitch 10.16mm 0.25W = 1/4W length 6.3mm diameter 2.5mm")
 		(property "Reference" "R13"
-			(at 5.08 -2.37 180)
+			(at 2.54 -3.175 -90)
 			(layer "F.SilkS")
 			(effects
@@
 		(tags "Resistor Axial_DIN0207 series Axial Horizontal pin pitch 10.16mm 0.25W = 1/4W length 6.3mm diameter 2.5mm")
 		(property "Reference" "R17"
-			(at 5.08 -2.37 0)
+			(at 12.03925 -0.011532 90)
 			(layer "F.SilkS")
 			(effects

Commit message: .
Parts:
- R1, R7: value 100 -> 68
- R13: value R_US -> 10K
- R17: value 560 -> 22K
- R18: value 330 -> 10K
- R2, R4: value 1.6 -> 68
- R3, R5: value R_US -> 68
Changed lines of the file:
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@@
 			)
 		)
-		(property "Value" "R_US"
+		(property "Value" "68"
 			(at 5.08 2.37 90)
 			(layer "F.Fab")
@@
 			)
 		)
-		(property "Value" "330"
+		(property "Value" "10K"
 			(at 5.08 2.37 0)
 			(layer "F.Fab")
@@
 			)
 		)
-		(property "Value" "100"
+		(property "Value" "68"
 			(at 5.08 2.37 90)
 			(layer "F.Fab")
@@
 			)
 		)
+		(sheetname "Raíz")
+		(sheetfile "PCB V1.kicad_sch")
 		(attr through_hole)
 		(fp_line
@@
 			(pintype "power_out")
 		)
-		(model "C:/Users/47698187/Downloads/ESP32-DEVKIT-V1--3DModel-STEP-269445.STEP"
+		(model "C:/Users/47698187/Documents/GitHub/Modelos-3D/Microcontroladores/ESP/ESP32/ESP32-DEVKIT-V1--3DModel-STEP-269445.STEP"
 			(offset
 				(xyz 14 -24.5 0)
@@
 			)
 		)
-		(property "Value" "R_US"
+		(property "Value" "68"
 			(at 5.08 2.37 90)
 			(layer "F.Fab")
@@
 			)
 		)
-		(property "Value" "1.6"
+		(property "Value" "68"
 			(at 5.08 2.37 90)
 			(layer "F.Fab")
@@
 			)
 		)
-		(model "C:/Users/47698187/Downloads/USB-B-S-S-B-TH-R.stp"
+		(model "C:/Users/47698187/Documents/GitHub/Modelos-3D/Conectores/USB/USB-B-S-S-B-TH-R.stp"
 			(offset
 				(xyz 7 -1.25 0)
@@
 			)
 		)
-		(property "Value" "100"
+		(property "Value" "68"
 			(at 5.08 2.37 90)
 			(layer "F.Fab")
@@
 			)
 		)
-		(property "Value" "1.6"
+		(property "Value" "68"
 			(at 5.08 2.37 90)
 			(layer "F.Fab")
@@
 			)
 		)
-		(property "Value" "R_US"
+		(property "Value" "10K"
 			(at 5.08 2.37 180)
 			(layer "F.Fab")
@@
 			)
 		)
-		(property "Value" "560"
+		(property "Value" "22K"
 			(at 5.08 2.37 0)
 			(layer "F.Fab")
