File: PCB/PCB V1/PCB V1.kicad_sch (KiCad schematic)
At the start: 50 parts, among them J1 Screw_Terminal_01x03, J2 Screw_Terminal_01x03, J3 USB_B, J4 Conn_01x02_Pin, K1 Relay_SPDT, K2 Relay_SPDT, Q1 S8050, Q2 S8050, Q3 S8050, SW1 On/Off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

Commit message: .
Parts:
- removed AHT1: AHT10, Connector_Molex:Molex_KK-254_AE-6410-04A_1x04_P2.54mm_Vertical, symbol Connector:Conn_01x04_Pin
- removed INA1: Sensor de Corriente, Connector_PinHeader_2.54mm:PinHeader_1x06_P2.54mm_Vertical, symbol Connector:Conn_01x06_Pin
- added DISPLAY2: AHT10, Connector_Molex:Molex_KK-254_AE-6410-04A_1x04_P2.54mm_Vertical, symbol Connector:Conn_01x04_Pin
- added DISPLAY3: DISPLAY, Connector_Molex:Molex_KK-254_AE-6410-04A_1x04_P2.54mm_Vertical, symbol Connector:Conn_01x04_Pin
- D5, D7: footprint Connector_Molex:Molex_KK-254_AE-6410-02A_1x02_P2.54mm_Vertical -> LED_THT:LED_D5.0mm_Clear
- J4: footprint Connector_PinHeader_2.54mm:PinHeader_1x02_P2.54mm_Vertical -> Connector_Molex:Molex_KK-254_AE-6410-02A_1x02_P2.54mm_Vertical
Connections:
- net +3.3V: now also DISPLAY2.2 (Pin_2), DISPLAY3.2 (Pin_2)
- net BOTON-A: now also ESP-1.16 (IO23); no longer ESP-1.9 (IO33)
- net BOTON-B: now also ESP-1.13 (IO39); no longer ESP-1.10 (IO32)
- net GND: now also DISPLAY2.1 (Pin_1), DISPLAY3.1 (Pin_1)
- net LED-A2: now also ESP-1.28 (IO15); no longer ESP-1.19 (IO3)
- net PUERTA: now also ESP-1.8 (IO25); no longer ESP-1.24 (IO17)
- net RELE-A: now also ESP-1.12 (IO34); no longer ESP-1.21 (IO19)
- net RELE-B: now also ESP-1.11 (IO35); no longer ESP-1.22 (IO18)
- net SCL: now also DISPLAY2.4 (Pin_4), DISPLAY3.4 (Pin_4)
- net SDA: now also DISPLAY2.3 (Pin_3), DISPLAY3.3 (Pin_3)

Commit message: .
Connections:
- net +5V: now also J2.2 (Pin_2), K2.11; no longer Cooler1.1 (Pin_1)
- net NO: now reaches J2.1 (Pin_1), K2.12
- net NO: now also Cooler1.1 (Pin_1)
Other:
- note added: "AHT10"
- note added: "BUZZER"
- note added: "COOLER"
- note added: "ESP32-DEVKIT-V1"
- note added: "INA219"
- note added: "LUCES DELANTERA"
- note added: "LUCES GUIÑO"
- note added: "USB B"
- moved on the sheet: D3, D4, D9, J3, R10, R4, R5, R9, SW1A, SW2, SW3

Commit message: .
Parts:
- removed D10: 1N4007, Diode_THT:D_DO-41_SOD81_P10.16mm_Horizontal, symbol Diode:1N4007
- R11: value 1.01K -> 22K
Connections:
- net +3.3V: no longer DISPLAY1.2 (Pin_2)
- net +5V: now also DISPLAY1.2 (Pin_2)
Changed lines of the file:
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@@
 	)
 	(junction
-		(at 193.04 76.2)
-		(diameter 0)
-		(color 0 0 0 0)
-	)
-	(junction
 		(at 66.04 118.11)
 		(diameter 0)
@@
 	)
 	(junction
-		(at 193.04 68.58)
-		(diameter 0)
-		(color 0 0 0 0)
-	)
-	(junction
 		(at 155.194 74.93)
 		(diameter 0)
@@
 	(wire
 		(pts
-			(xy 193.04 74.93) (xy 193.04 76.2)
+			(xy 193.04 74.93) (xy 193.04 78.74)
 		)
 		(stroke
@@
 	(wire
 		(pts
-			(xy 193.04 76.2) (xy 193.04 78.74)
-		)
-		(stroke
-			(width 0)
-			(type default)
-		)
-	)
-	(wire
-		(pts
-			(xy 193.04 76.2) (xy 201.93 76.2)
-		)
-		(stroke
-			(width 0)
-			(type default)
-		)
-	)
-	(wire
-		(pts
 			(xy 120.65 101.6) (xy 120.65 104.14)
 		)
@@
 	(wire
 		(pts
-			(xy 193.04 68.58) (xy 201.93 68.58)
-		)
-		(stroke
-			(width 0)
-			(type default)
-		)
-	)
-	(wire
-		(pts
 			(xy 54.61 82.55) (xy 53.34 82.55)
 		)
@@
 	(wire
 		(pts
-			(xy 193.04 67.31) (xy 193.04 68.58)
-		)
-		(stroke
-			(width 0)
-			(type default)
-		)
-	)
-	(wire
-		(pts
 			(xy 69.85 102.87) (xy 69.85 101.6)
 		)
@@
 	(wire
 		(pts
-			(xy 193.04 68.58) (xy 193.04 69.85)
+			(xy 193.04 67.31) (xy 193.04 69.85)
 		)
 		(stroke
@@
 	)
 	(symbol
-		(lib_id "Diode:1N4007")
-		(at 201.93 72.39 270)
-		(unit 1)
-		(exclude_from_sim no)
-		(in_bom yes)
-		(on_board yes)
-		(dnp no)
-		(fields_autoplaced yes)
-		(property "Reference" "D10"
-			(at 204.47 71.1199 90)
-			(effects
-				(font
-					(size 1.27 1.27)
-				)
-				(justify left)
-			)
-		)
-		(property "Value" "1N4007"
-			(at 204.47 73.6599 90)
-			(effects
-				(font
-					(size 1.27 1.27)
-				)
-				(justify left)
-			)
-		)
-		(property "Footprint" "Diode_THT:D_DO-41_SOD81_P10.16mm_Horizontal"
-			(at 197.485 72.39 0)
-			(effects
-				(font
-					(size 1.27 1.27)
-				)
-				(hide yes)
-			)
-		)
-		(property "Datasheet" "http://www.vishay.com/docs/88503/1n4001.pdf"
-			(at 201.93 72.39 0)
-			(effects
-				(font
-					(size 1.27 1.27)
-				)
-				(hide yes)
-			)
-		)
-		(property "Description" "1000V 1A General Purpose Rectifier Diode, DO-41"
-			(at 201.93 72.39 0)
-			(effects
-				(font
-					(size 1.27 1.27)
-				)
-				(hide yes)
-			)
-		)
-		(property "Sim.Device" "D"
-			(at 201.93 72.39 0)
-			(effects
-				(font
-					(size 1.27 1.27)
-				)
-				(hide yes)
-			)
-		)
-		(property "Sim.Pins" "1=K 2=A"
-			(at 201.93 72.39 0)
-			(effects
-				(font
-					(size 1.27 1.27)
-				)
-				(hide yes)
-			)
-		)
-		(pin "2"
-		)
-		(pin "1"
-		)
-		(instances
-			(project "PCB V1"
-				(path "/9d3c0d60-bbc5-4e33-843b-0a3b234644e7"
-					(reference "D10")
-					(unit 1)
-				)
-			)
-		)
-	)
-	(symbol
 		(lib_id "power:GND")
 		(at 242.57 80.01 0)
@@
 	)
 	(symbol
-		(lib_id "power:+3.3V")
-		(at 201.93 31.75 0)
-		(unit 1)
-		(exclude_from_sim no)
-		(in_bom yes)
-		(on_board yes)
-		(dnp no)
-		(property "Reference" "#PWR033"
-			(at 201.93 35.56 0)
-			(effects
-				(font
-					(size 1.27 1.27)
-				)
-				(hide yes)
-			)
-		)
-		(property "Value" "+3.3V"
-			(at 200.66 27.94 0)
-			(effects
-				(font
-					(size 1.27 1.27)
-				)
-			)
-		)
-		(property "Footprint" ""
-			(at 201.93 31.75 0)
-			(effects
-				(font
-					(size 1.27 1.27)
-				)
-				(hide yes)
-			)
-		)
-		(property "Datasheet" ""
-			(at 201.93 31.75 0)
-			(effects
-				(font
-					(size 1.27 1.27)
-				)
-				(hide yes)
-			)
-		)
-		(property "Description" "Power symbol creates a global label with name \"+3.3V\""
-			(at 201.93 31.75 0)
-			(effects
-				(font
-					(size 1.27 1.27)
-				)
-				(hide yes)
-			)
-		)
-		(pin "1"
-		)
-		(instances
-			(project "PCB V1"
-				(path "/9d3c0d60-bbc5-4e33-843b-0a3b234644e7"
-					(reference "#PWR033")
-					(unit 1)
-				)
-			)
-		)
-	)
-	(symbol
 		(lib_id "Transistor_BJT:S8050")
 		(at 67.31 132.08 0)
@@
 	)
 	(symbol
+		(lib_id "power:+5V")
+		(at 201.93 31.75 0)
+		(unit 1)
+		(exclude_from_sim no)
+		(in_bom yes)
+		(on_board yes)
+		(dnp no)
+		(property "Reference" "#PWR04"
+			(at 201.93 35.56 0)
+			(effects
+				(font
+					(size 1.27 1.27)
+				)
+				(hide yes)
+			)
+		)
+		(property "Value" "+5V"
+			(at 201.93 33.02 0)
+			(effects
+				(font
+					(size 1.27 1.27)
+				)
+			)
+		)
+		(property "Footprint" ""
+			(at 201.93 31.75 0)
+			(effects
+				(font
+					(size 1.27 1.27)
+				)
+				(hide yes)
+			)
+		)
+		(property "Datasheet" ""
+			(at 201.93 31.75 0)
+			(effects
+				(font
+					(size 1.27 1.27)
+				)
+				(hide yes)
+			)
+		)
+		(property "Description" "Power symbol creates a global label with name \"+5V\""
+			(at 201.93 31.75 0)
+			(effects
+				(font
+					(size 1.27 1.27)
+				)
+				(hide yes)
+			)
+		)
+		(pin "1"
+		)
+		(instances
+			(project "PCB V1"
+				(path "/9d3c0d60-bbc5-4e33-843b-0a3b234644e7"
+					(reference "#PWR04")
+					(unit 1)
+				)
+			)
+		)
+	)
+	(symbol
 		(lib_id "Connector:Conn_01x04_Pin")
 		(at 152.5503 28.535 0)
@@
 			)
 		)
-		(property "Value" "1.01K"
-			(at 180.086 88.138 0)
+		(property "Value" "22K"
+			(at 186.69 88.9 0)
 			(effects
 				(font

Commit message: .
Parts:
- removed D9: 1N4007, Diode_THT:D_DO-41_SOD81_P10.16mm_Horizontal, symbol Diode:1N4007
- added C?: 100uf, Capacitor_THT:C_Disc_D7.5mm_W4.4mm_P5.00mm, symbol Device:C
- added C?: 100uF, Capacitor_THT:CP_Radial_D10.0mm_P3.50mm, symbol Device:C_Polarized
- added C?: 10uF, Capacitor_THT:CP_Radial_D5.0mm_P2.50mm, symbol Device:C_Polarized
- added Cooler?: Bornera Cooler, TerminalBlock:TerminalBlock_bornier-2_P5.08mm, symbol Connector:Screw_Terminal_01x02
- added D?: 1N4007, Diode_THT:D_DO-41_SOD81_P10.16mm_Horizontal, symbol Diode:1N4007
- added R?: 560, Resistor_THT:R_Axial_DIN0207_L6.3mm_D2.5mm_P10.16mm_Horizontal, symbol Device:R_US
- added R?: 330, Resistor_THT:R_Axial_DIN0207_L6.3mm_D2.5mm_P10.16mm_Horizontal, symbol Device:R_US
- added U?: LM317_TO-220, Package_TO_SOT_THT:TO-220F-3_Vertical, symbol Regulator_Linear:LM317_TO-220
Connections:
- net +3.3V: now also D5.2 (A)
- net +5V: no longer J2.2 (Pin_2), K2.11
- net GND: now also C?.2, C?.2, C?.2, Cooler?.1 (Pin_1), R?.2; no longer R1.2
- net NO: no longer Cooler1.1 (Pin_1)
- net RELE-B: no longer D5.2 (A)
- net at D6.2 (A), K1.A2, Q1.3 (C): now also R1.2
- net +5VANTESDELLAVE: now reaches SW1.1 (A)
- net +5VANTESDELLAVE: now also J3.1 (VBUS), D?.1 (K)
- new net: R?.1, R?.1, U?.1 (ADJ)
- new net: C?.1, C?.1, D?.2 (A), R?.2, U?.2 (VO)
- new net: J2.2 (Pin_2), K2.11
- new net +12V: C?.1, Cooler?.2 (Pin_2), U?.3 (VI)
- new net 5V: Cooler1.1 (Pin_1)
Other:
- moved on the sheet: D5

Commit message: .
Parts:
- Cooler2: renamed from Cooler?; value Bornera Cooler -> Bateria
- R1, R7: value R_US -> 100
- R10, R9: value R_US -> 10K
- R12: value R_LDR -> 10K
- R2, R4: value R_US -> 1.6
- SW1: footprint Button_Switch_THT:SW_Slide_SPDT_Straight_CK_OS102011MS2Q -> TerminalBlock:TerminalBlock_bornier-2_P5.08mm
- gave numbers to parts that had none: 7
Connections:
- net 5V is gone; now on net +5V: Cooler1.1 (Pin_1)
- net +3.3V: now also D7.2 (A)
- net +5VANTESDELLAVE: now also C6.1
- net GND: no longer R7.2
- net RELE-A: no longer D7.2 (A)
- net at C5.1, D9.2 (A), R18.2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: no longer C6.1
- net at D8.2 (A), K2.A2, Q2.3 (C): now also R7.2
Other:
- moved on the sheet: D9

Commit message: .
Parts:
- added D10: 1N4007, Diode_THT:D_DO-41_SOD81_P10.16mm_Horizontal, symbol Diode:1N4007
Connections:
- net +5VANTESDELLAVE: now also D10.1 (K); no longer J3.1 (VBUS)
- net BOTON-B: now also ESP-1.21 (IO19); no longer ESP-1.13 (IO39)
- net BUZZER: now also ESP-1.7 (IO26); no longer ESP-1.23 (IO5)
- net LED-A1: now also ESP-1.24 (IO17); no longer ESP-1.18 (IO1)
- net LED-A2: now also ESP-1.23 (IO5); no longer ESP-1.28 (IO15)
- net LED-B1: now also ESP-1.28 (IO15); no longer ESP-1.27 (IO2)
- net PUERTA: now also ESP-1.22 (IO18); no longer ESP-1.8 (IO25)
- new net: D10.2 (A), J3.1 (VBUS)
Changed lines of the file:
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@@
 	)
 	(junction
-		(at 265.43 65.0001)
+		(at 163.83 105.41)
 		(diameter 0)
 		(color 0 0 0 0)
 	)
 	(junction
-		(at 160.02 105.41)
+		(at 265.43 65.0001)
 		(diameter 0)
 		(color 0 0 0 0)
@@
 	(wire
 		(pts
-			(xy 160.02 105.41) (xy 156.21 105.41)
-		)
-		(stroke
-			(width 0)
-			(type default)
-		)
-	)
-	(wire
-		(pts
-			(xy 160.02 105.41) (xy 163.83 105.41)
-		)
-		(stroke
-			(width 0)
-			(type default)
-		)
-	)
-	(wire
-		(pts
 			(xy 81.28 36.83) (xy 82.55 36.83)
 		)
@@
 	(wire
 		(pts
-			(xy 160.02 104.14) (xy 160.02 105.41)
-		)
-		(stroke
-			(width 0)
-			(type default)
-		)
-	)
-	(wire
-		(pts
 			(xy 166.5203 31.075) (xy 165.2503 31.075)
 		)
@@
 		)
 	)
-	(global_label "BUZZER"
-		(shape input)
-		(at 82.55 55.88 180)
-		(fields_autoplaced yes)
-		(effects
-			(font
-				(size 1.27 1.27)
-			)
-			(justify right)
-		)
-		(property "Intersheetrefs" "${INTERSHEET_REFS}"
-			(at 72.1263 55.88 0)
-			(effects
-				(font
-					(size 1.27 1.27)
-				)
-				(justify right)
-				(hide yes)
-			)
-		)
-	)
 	(global_label "SDA"
 		(shape input)
@@
 		)
 	)
-	(global_label "LED-A1"
-		(shape input)
-		(at 82.55 45.72 180)
-		(fields_autoplaced yes)
-		(effects
-			(font
-				(size 1.27 1.27)
-			)
-			(justify right)
-		)
-		(property "Intersheetrefs" "${INTERSHEET_REFS}"
-			(at 72.2472 45.72 0)
-			(effects
-				(font
-					(size 1.27 1.27)
-				)
-				(justify right)
-				(hide yes)
-			)
-		)
-	)
 	(global_label "RELE-A"
 		(shape input)
@@
 		)
 	)
-	(global_label "LED-A2"
+	(global_label "BOTON-B"
 		(shape input)
-		(at 82.55 66.04 180)
+		(at 82.55 76.2 180)
 		(fields_autoplaced yes)
 		(effects
@@
 		)
 		(property "Intersheetrefs" "${INTERSHEET_REFS}"
-			(at 72.2472 66.04 0)
+			(at 70.4933 76.2 0)
 			(effects
 				(font
@@
 		)
 	)
-	(global_label "SCL"
+	(global_label "BUZZER"
 		(shape input)
-		(at 193.04 34.29 0)
+		(at 120.65 55.88 0)
 		(fields_autoplaced yes)
 		(effects
@@
 		)
 		(property "Intersheetrefs" "${INTERSHEET_REFS}"
-			(at 199.5328 34.29 0)
+			(at 131.0737 55.88 0)
 			(effects
 				(font
@@
 	(global_label "SCL"
 		(shape input)
-		(at 157.6303 33.615 0)
+		(at 193.04 34.29 0)
 		(fields_autoplaced yes)
 		(effects
@@
 		)
 		(property "Intersheetrefs" "${INTERSHEET_REFS}"
-			(at 164.1231 33.615 0)
+			(at 199.5328 34.29 0)
 			(effects
 				(font
@@
 		)
 	)
-	(global_label "PUERTA"
+	(global_label "SCL"
 		(shape input)
-		(at 120.65 53.34 0)
+		(at 157.6303 33.615 0)
 		(fields_autoplaced yes)
 		(effects
@@
 		)
 		(property "Intersheetrefs" "${INTERSHEET_REFS}"
-			(at 130.7109 53.34 0)
+			(at 164.1231 33.615 0)
 			(effects
 				(font
@@
 		)
 	)
-	(global_label "LED-B1"
-		(shape input)
-		(at 82.55 48.26 180)
-		(fields_autoplaced yes)
-		(effects
-			(font
-				(size 1.27 1.27)
-			)
-			(justify right)
-		)
-		(property "Intersheetrefs" "${INTERSHEET_REFS}"
-			(at 72.0658 48.26 0)
-			(effects
-				(font
-					(size 1.27 1.27)
-				)
-				(justify right)
-				(hide yes)
-			)
-		)
-	)
 	(global_label "LDR"
 		(shape input)
@@
 		)
 	)
-	(global_label "LED-A1"
+	(global_label "LED-B1"
 		(shape input)
-		(at 33.02 53.34 180)
+		(at 82.55 66.04 180)
 		(fields_autoplaced yes)
 		(effects
@@
 		)
 		(property "Intersheetrefs" "${INTERSHEET_REFS}"
-			(at 22.7172 53.34 0)
+			(at 72.0658 66.04 0)
 			(effects
 				(font
@@
 		)
 	)
-	(global_label "BUZZER"
+	(global_label "LED-A1"
 		(shape input)
-		(at 185.42 91.44 270)
+		(at 33.02 53.34 180)
 		(fields_autoplaced yes)
 		(effects
@@
 		)
 		(property "Intersheetrefs" "${INTERSHEET_REFS}"
-			(at 185.42 101.8637 90)
+			(at 22.7172 53.34 0)
 			(effects
 				(font
@@
 		)
 	)
-	(global_label "BOTON-B"
+	(global_label "BUZZER"
 		(shape input)
-		(at 120.65 73.66 0)
+		(at 185.42 91.44 270)
 		(fields_autoplaced yes)
 		(effects
@@
 				(size 1.27 1.27)
 			)
-			(justify left)
+			(justify right)
 		)
 		(property "Intersheetrefs" "${INTERSHEET_REFS}"
-			(at 132.7067 73.66 0)
+			(at 185.42 101.8637 90)
 			(effects
 				(font
 					(size 1.27 1.27)
 				)
-				(justify left)
+				(justify right)
 				(hide yes)
 			)
@@
 		)
 	)
+	(global_label "LED-A1"
+		(shape input)
+		(at 82.55 71.12 180)
+		(fields_autoplaced yes)
+		(effects
+			(font
+				(size 1.27 1.27)
+			)
+			(justify right)
+		)
+		(property "Intersheetrefs" "${INTERSHEET_REFS}"
+			(at 72.2472 71.12 0)
+			(effects
+				(font
+					(size 1.27 1.27)
+				)
+				(justify right)
+				(hide yes)
+			)
+		)
+	)
 	(global_label "RELE-B"
 		(shape input)
@@
 		)
 	)
+	(global_label "LED-A2"
+		(shape input)
+		(at 82.55 55.88 180)
+		(fields_autoplaced yes)
+		(effects
+			(font
+				(size 1.27 1.27)
+			)
+			(justify right)
+		)
+		(property "Intersheetrefs" "${INTERSHEET_REFS}"
+			(at 72.2472 55.88 0)
+			(effects
+				(font
+					(size 1.27 1.27)
+				)
+				(justify right)
+				(hide yes)
+			)
+		)
+	)
 	(global_label "RELE-A"
 		(shape input)
@@
 		)
 	)
+	(global_label "PUERTA"
+		(shape input)
+		(at 82.55 73.66 180)
+		(fields_autoplaced yes)
+		(effects
+			(font
+				(size 1.27 1.27)
+			)
+			(justify right)
+		)
+		(property "Intersheetrefs" "${INTERSHEET_REFS}"
+			(at 72.4891 73.66 0)
+			(effects
+				(font
+					(size 1.27 1.27)
+				)
+				(justify right)
+				(hide yes)
+			)
+		)
+	)
 	(global_label "LED-B2"
 		(shape input)
@@
 	(symbol
 		(lib_id "power:+5V")
-		(at 160.02 104.14 0)
+		(at 163.83 105.41 0)
 		(unit 1)
 		(exclude_from_sim no)
@@
 		(fields_autoplaced yes)
 		(property "Reference" "#PWR041"
-			(at 160.02 107.95 0)
+			(at 163.83 109.22 0)
 			(effects
 				(font
@@
 		)
 		(property "Value" "+5VANTESDELLAVE"
-			(at 160.02 99.06 0)
+			(at 163.83 100.33 0)
 			(effects
 				(font
@@
 		)
 		(property "Footprint" ""
-			(at 160.02 104.14 0)
+			(at 163.83 105.41 0)
 			(effects
 				(font
@@
 		)
 		(property "Datasheet" ""
-			(at 160.02 104.14 0)
+			(at 163.83 105.41 0)
 			(effects
 				(font
@@
 		)
 		(property "Description" "Power symbol creates a global label with name \"+5V\""
-			(at 160.02 104.14 0)
+			(at 163.83 105.41 0)
 			(effects
 				(font
@@
 					(unit 1)
 				)
+			)
+		)
+	)
+	(symbol
+		(lib_id "Diode:1N4007")
+		(at 160.02 105.41 180)
+		(unit 1)
+		(exclude_from_sim no)
+		(in_bom yes)
+		(on_board yes)
+		(dnp no)
+		(property "Reference" "D10"
+			(at 160.528 107.696 0)
+			(effects
+				(font
+					(size 1.27 1.27)
+				)
+			)
+		)
+		(property "Value" "1N4007"
+			(at 160.528 109.474 0)
+			(effects
+				(font
+					(size 1.27 1.27)
+				)
+			)
+		)
+		(property "Footprint" "Diode_THT:D_DO-41_SOD81_P10.16mm_Horizontal"
+			(at 160.02 100.965 0)
+			(effects
+				(font
+					(size 1.27 1.27)
+				)
+				(hide yes)
+			)
+		)
+		(property "Datasheet" "http://www.vishay.com/docs/88503/1n4001.pdf"
+			(at 160.02 105.41 0)
+			(effects
+				(font
+					(size 1.27 1.27)
+				)
+				(hide yes)
+			)
+		)
+		(property "Description" "1000V 1A General Purpose Rectifier Diode, DO-41"
+			(at 160.02 105.41 0)
+			(effects
+				(font
+					(size 1.27 1.27)
+				)
+				(hide yes)
+			)
+		)
+		(property "Sim.Device" "D"
+			(at 160.02 105.41 0)
+			(effects
+				(font
+					(size 1.27 1.27)
+				)
+				(hide yes)
+			)
+		)
+		(property "Sim.Pins" "1=K 2=A"
+			(at 160.02 105.41 0)
+			(effects
+				(font
+					(size 1.27 1.27)
+				)
+				(hide yes)
+			)
+		)
+		(pin "2"
+		)
+		(pin "1"
+		)
+		(instances
+			(project ""
+				(path "/9d3c0d60-bbc5-4e33-843b-0a3b234644e7"
+					(reference "D10")
+					(unit 1)
+				)
