File: PCB/PCB V1/PCB V1.kicad_sch (KiCad schematic)
At the start: 57 parts, among them J1 Screw_Terminal_01x03, J2 Screw_Terminal_01x03, J3 USB_B, J4 Conn_01x02_Pin, K1 Relay_SPDT, K2 Relay_SPDT, Q1 S8050, Q2 S8050, Q3 S8050, SW1 On/Off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

Commit message: .
Parts:
- U1, U2: footprint Package_TO_SOT_THT:TO-220F-3_Vertical -> Package_TO_SOT_THT:TO-92_Inline
Connections:
- net LDR: now also ESP-1.11 (IO35); no longer ESP-1.14 (IO36)
Changed lines of the file:
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@@
 		(exclude_from_sim no)
 		(at 180.34 38.1 0)
-		(size 31.75 21.59)
+		(size 33.02 21.59)
 		(stroke
 			(width 0)
@@
 	(global_label "LDR"
 		(shape input)
-		(at 120.65 71.12 0)
+		(at 120.65 68.58 0)
 		(fields_autoplaced yes)
 		(effects
@@
 		)
 		(property "Intersheetrefs" "${INTERSHEET_REFS}"
-			(at 127.2033 71.12 0)
+			(at 127.2033 68.58 0)
 			(effects
 				(font
@@
 		)
 		(property "Value" "10K"
-			(at 188.722 49.276 90)
+			(at 190.5 49.53 90)
 			(effects
 				(font
@@
 			)
 		)
-		(property "Footprint" "Package_TO_SOT_THT:TO-220F-3_Vertical"
+		(property "Footprint" "Package_TO_SOT_THT:TO-92_Inline"
 			(at 237.49 58.42 0)
 			(effects
@@
 			)
 		)
-		(property "Footprint" "Package_TO_SOT_THT:TO-220F-3_Vertical"
+		(property "Footprint" "Package_TO_SOT_THT:TO-92_Inline"
 			(at 237.49 88.9 0)
 			(effects

Commit message: .
Connections:
- net BOTON-B: now also ESP-1.7 (IO26); no longer ESP-1.21 (IO19)
- net BUZZER: now also ESP-1.21 (IO19); no longer ESP-1.7 (IO26)
- net LED-A1: now also ESP-1.25 (IO16); no longer ESP-1.24 (IO17)
- net LED-B1: now also ESP-1.24 (IO17); no longer ESP-1.28 (IO15)
- net LED-B2: now also ESP-1.22 (IO18); no longer ESP-1.26 (IO4)
- net PUERTA: now also ESP-1.26 (IO4); no longer ESP-1.22 (IO18)
- net RELE-A: now also ESP-1.13 (IO39); no longer ESP-1.12 (IO34)
- net RELE-B: now also ESP-1.12 (IO34); no longer ESP-1.13 (IO39)

Commit message: .
Connections:
- net BOTON-A: now also ESP-1.10 (IO32); no longer ESP-1.16 (IO23)
- net BOTON-B: now also ESP-1.9 (IO33); no longer ESP-1.7 (IO26)
- net PUERTA: now also ESP-1.7 (IO26); no longer ESP-1.26 (IO4)

Commit message: .
Connections:
- net NO: no longer names the net of J2.1 (Pin_1), K2.12
Other:
- moved on the sheet: C4, C5, C6, D9, R17, R18, U2

Commit message: .
Parts:
- removed D10: 1N4007, Diode_THT:D_DO-41_SOD81_P10.16mm_Horizontal, symbol Diode:1N4007
Connections:
- net +5VANTESDELLAVE: now also J3.1 (VBUS)
Changed lines of the file:
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@@
 	)
 	(junction
-		(at 163.83 105.41)
+		(at 265.43 65.0001)
 		(diameter 0)
 		(color 0 0 0 0)
 	)
 	(junction
-		(at 265.43 65.0001)
+		(at 267.97 95.25)
 		(diameter 0)
 		(color 0 0 0 0)
 	)
 	(junction
-		(at 267.97 95.25)
+		(at 163.83 105.41)
 		(diameter 0)
 		(color 0 0 0 0)
@@
 	(wire
 		(pts
+			(xy 156.21 105.41) (xy 163.83 105.41)
+		)
+		(stroke
+			(width 0)
+			(type default)
+		)
+	)
+	(wire
+		(pts
 			(xy 187.96 74.93) (xy 193.04 74.93)
 		)
@@
 					(unit 1)
 				)
-			)
-		)
-	)
-	(symbol
-		(lib_id "Diode:1N4007")
-		(at 160.02 105.41 180)
-		(unit 1)
-		(exclude_from_sim no)
-		(in_bom yes)
-		(on_board yes)
-		(dnp no)
-		(property "Reference" "D10"
-			(at 160.528 107.696 0)
-			(effects
-				(font
-					(size 1.27 1.27)
-				)
-			)
-		)
-		(property "Value" "1N4007"
-			(at 160.528 109.474 0)
-			(effects
-				(font
-					(size 1.27 1.27)
-				)
-			)
-		)
-		(property "Footprint" "Diode_THT:D_DO-41_SOD81_P10.16mm_Horizontal"
-			(at 160.02 100.965 0)
-			(effects
-				(font
-					(size 1.27 1.27)
-				)
-				(hide yes)
-			)
-		)
-		(property "Datasheet" "http://www.vishay.com/docs/88503/1n4001.pdf"
-			(at 160.02 105.41 0)
-			(effects
-				(font
-					(size 1.27 1.27)
-				)
-				(hide yes)
-			)
-		)
-		(property "Description" "1000V 1A General Purpose Rectifier Diode, DO-41"
-			(at 160.02 105.41 0)
-			(effects
-				(font
-					(size 1.27 1.27)
-				)
-				(hide yes)
-			)
-		)
-		(property "Sim.Device" "D"
-			(at 160.02 105.41 0)
-			(effects
-				(font
-					(size 1.27 1.27)
-				)
-				(hide yes)
-			)
-		)
-		(property "Sim.Pins" "1=K 2=A"
-			(at 160.02 105.41 0)
-			(effects
-				(font
-					(size 1.27 1.27)
-				)
-				(hide yes)
-			)
-		)
-		(pin "2"
-		)
-		(pin "1"
-		)
-		(instances
-			(project "PCB V1"
-				(path "/9d3c0d60-bbc5-4e33-843b-0a3b234644e7"
-					(reference "D10")
-					(unit 1)
-				)

Commit message: .
Parts:
- R13: value R_US -> 10K
- R17: value 560 -> 22K
- R18: value 330 -> 10K
- R2, R4: value 1.6 -> 68
- R3, R5: value R_US -> 68
Changed lines of the file:
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@@
 		)
 	)
-	(text_box "DISPLAY IDC"
+	(text_box "DISPLAY LCD"
 		(exclude_from_sim no)
 		(at 180.34 20.32 0)
@@
 			)
 		)
-		(property "Value" "560"
+		(property "Value" "22K"
 			(at 238.76 107.95 0)
 			(effects
@@
 			)
 		)
-		(property "Value" "1.6"
+		(property "Value" "68"
 			(at 48.2601 77.47 90)
 			(effects
@@
 			)
 		)
-		(property "Value" "1.6"
+		(property "Value" "68"
 			(at 43.1801 55.88 90)
 			(effects
@@
 		(on_board yes)
 		(dnp no)
-		(fields_autoplaced yes)
 		(property "Reference" "R13"
-			(at 191.516 109.2199 0)
+			(at 196.85 109.2199 0)
 			(effects
 				(font
 					(size 1.27 1.27)
 				)
-				(justify left)
+				(justify right)
 			)
 		)
-		(property "Value" "R_US"
-			(at 191.516 111.7599 0)
+		(property "Value" "10K"
+			(at 191.77 108.712 90)
 			(effects
 				(font
 					(size 1.27 1.27)
 				)
-				(justify left)
+				(justify right)
 			)
 		)
@@
 			)
 		)
-		(property "Value" "R_US"
+		(property "Value" "68"
 			(at 43.1801 63.5 90)
 			(effects
@@
 			)
 		)
-		(property "Value" "R_US"
+		(property "Value" "68"
 			(at 48.2601 85.09 90)
 			(effects
@@
 			)
 		)
-		(property "Value" "330"
+		(property "Value" "10K"
 			(at 252.73 96.52 0)
 			(effects

Commit message: .
Parts:
- R1, R7: value 100 -> 68
Changed lines of the file:
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@@
 			)
 		)
-		(property "Value" "100"
+		(property "Value" "68"
 			(at 31.75 115.57 0)
 			(effects
@@
 		(dnp no)
 		(property "Reference" "R7"
-			(at 95.25 115.57 90)
+			(at 85.09 114.3 0)
 			(effects
 				(font
 					(size 1.27 1.27)
 				)
-				(hide yes)
 			)
 		)
-		(property "Value" "100"
+		(property "Value" "68"
 			(at 83.82 115.57 0)
 			(effects
