File: PCB/PCB V1/PCB V1.kicad_sch (KiCad schematic)
At the start: 56 parts, among them J1 Screw_Terminal_01x03, J2 Screw_Terminal_01x03, J3 USB_B, J4 Conn_01x02_Pin, K1 Relay_SPDT, K2 Relay_SPDT, Q1 S8050, Q2 S8050, Q3 S8050, SW1 On/Off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

Commit message: .
Connections:
- net RELE-A: now also ESP-1.5 (IO14); no longer ESP-1.13 (IO39)
- net RELE-B: now also ESP-1.6 (IO27); no longer ESP-1.12 (IO34)
