File: PCB/PCB V1/_autosave-PCB V1.kicad_pcb (KiCad board)
At the start: 2 copper layers, 100 x 100 mm, 55 parts, among them J1 Screw_Terminal_01x03, J2 Screw_Terminal_01x03, J3 USB_B, J4 Conn_01x02_Pin, K1 Relay_SPDT, K2 Relay_SPDT, Q1 S8050, Q2 S8050, Q3 S8050, SW1 On/Off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

Commit message: .
Connections:
- ESP-1 pad 11: unconnected-(ESP-1-IO35-Pad11) -> LDR
- ESP-1 pad 14: LDR -> unconnected-(ESP-1-IO36-Pad14)
Routing:
- net LDR: track 19.1 -> 22.6 mm
Changed lines of the file:
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@@
 	(net 48 "+5VANTESDELLAVE")
 	(net 49 "Net-(J2-Pin_2)")
-	(net 50 "unconnected-(ESP-1-IO35-Pad11)")
+	(net 50 "unconnected-(ESP-1-IO36-Pad14)")
 	(net 51 "Net-(U2-ADJ)")
 	(net 52 "Net-(D10-A)")
@@
 		(tags "terminal block bornier3")
 		(property "Reference" "J2"
-			(at 5.05 -4.65 270)
+			(at 5.05 -4.65 -90)
 			(layer "F.SilkS")
 			(effects
@@
 		)
 		(property "Value" "Screw_Terminal_01x03"
-			(at 5.08 5.08 270)
+			(at 5.08 5.08 -90)
 			(layer "F.Fab")
 			(effects
@@
 		)
 		(fp_text user "${REFERENCE}"
-			(at 5.08 0 270)
+			(at 5.08 0 -90)
 			(layer "F.Fab")
 			(effects
@@
 		(tags "Resistor Axial_DIN0207 series Axial Horizontal pin pitch 10.16mm 0.25W = 1/4W length 6.3mm diameter 2.5mm")
 		(property "Reference" "R1"
-			(at 5.08 -2.37 360)
+			(at 5.08 -2.37 0)
 			(layer "F.SilkS")
 			(effects
@@
 		)
 		(property "Value" "100"
-			(at 5.08 2.37 360)
+			(at 5.08 2.37 0)
 			(layer "F.Fab")
 			(effects
@@
 		)
 		(fp_text user "${REFERENCE}"
-			(at 5.08 0 360)
+			(at 5.08 0 0)
 			(layer "F.Fab")
 			(effects
@@
 		(tags "terminal block bornier3")
 		(property "Reference" "J1"
-			(at 5.05 -4.65 270)
+			(at 5.05 -4.65 -90)
 			(layer "F.SilkS")
 			(effects
@@
 		)
 		(property "Value" "Screw_Terminal_01x03"
-			(at 5.08 5.08 270)
+			(at 5.08 5.08 -90)
 			(layer "F.Fab")
 			(effects
@@
 		)
 		(fp_text user "${REFERENCE}"
-			(at 5.08 0 270)
+			(at 5.08 0 -90)
 			(layer "F.Fab")
 			(effects
@@
 			(layers "*.Cu" "*.Mask")
 			(remove_unused_layers no)
-			(net 50 "unconnected-(ESP-1-IO35-Pad11)")
+			(net 31 "LDR")
 			(pinfunction "IO35")
 			(pintype "bidirectional")
@@
 			(layers "*.Cu" "*.Mask")
 			(remove_unused_layers no)
-			(net 31 "LDR")
+			(net 50 "unconnected-(ESP-1-IO36-Pad14)")
 			(pinfunction "IO36")
 			(pintype "bidirectional")
@@
 	)
 	(segment
-		(start 156.895 100.731042)
-		(end 155.623958 99.46)
+		(start 155.623958 99.46)
+		(end 154.5 99.46)
 		(width 1)
 		(layer "B.Cu")
@@
 	)
 	(segment
-		(start 155.623958 99.46)
-		(end 154.5 99.46)
+		(start 156.928958 100.731042)
+		(end 162.66 95)
 		(width 1)
 		(layer "B.Cu")
@@
 	)
 	(segment
-		(start 155.04 98.92)
-		(end 155.04 95)
+		(start 152.5 110.42)
+		(end 156.895 106.025)
 		(width 1)
 		(layer "B.Cu")
@@
 	)
 	(segment
-		(start 154.5 99.46)
-		(end 155.04 98.92)
+		(start 156.351979 100.188021)
+		(end 155.623958 99.46)
 		(width 1)
 		(layer "B.Cu")
@@
 	)
 	(segment
-		(start 152.5 110.42)
-		(end 156.895 106.025)
+		(start 156.895 106.025)
+		(end 156.895 100.731042)
 		(width 1)
 		(layer "B.Cu")
@@
 	)
 	(segment
-		(start 156.895 106.025)
+		(start 156.351979 100.188021)
 		(end 156.895 100.731042)
 		(width 1)
 		(layer "B.Cu")
+		(net 31)
+	)
+	(segment
+		(start 156.895 100.731042)
+		(end 156.928958 100.731042)
+		(width 1)
+		(layer "B.Cu")
