File: PCB/PCB V1/_autosave-PCB V1.kicad_sch (KiCad schematic)
At the start: 57 parts, among them J1 Screw_Terminal_01x03, J2 Screw_Terminal_01x03, J3 USB_B, J4 Conn_01x02_Pin, K1 Relay_SPDT, K2 Relay_SPDT, Q1 S8050, Q2 S8050, Q3 S8050, SW1 On/Off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

Commit message: .
Connections:
- net LDR: now also ESP-1.11 (IO35); no longer ESP-1.14 (IO36)
Changed lines of the file:
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@@
 		(exclude_from_sim no)
 		(at 180.34 38.1 0)
-		(size 31.75 21.59)
+		(size 33.02 21.59)
 		(stroke
 			(width 0)
@@
 	(global_label "LDR"
 		(shape input)
-		(at 120.65 71.12 0)
+		(at 120.65 68.58 0)
 		(fields_autoplaced yes)
 		(effects
@@
 		)
 		(property "Intersheetrefs" "${INTERSHEET_REFS}"
-			(at 127.2033 71.12 0)
+			(at 127.2033 68.58 0)
 			(effects
 				(font
@@
 		)
 		(property "Value" "10K"
-			(at 188.722 49.276 90)
-			(effects
-				(font
+			(at 190.5 49.53 90)
+			(effects
+				(font
